Commit message: Initial push of SLAM and AMCL for Robot

File: robot_model_pkg/urdf/gazebo_control.xacro (robot description, xacro)
@@ -6,5 +6,5 @@
             <left_joint>left_wheel_joint</left_joint>
             <right_joint>right_wheel_joint</right_joint>
-            <wheel_separation>0.188</wheel_separation>
+            <wheel_separation>0.193</wheel_separation>
             <wheel_diameter>0.43</wheel_diameter>
             <!-- Limits -->

File: robot_model_pkg/urdf/lidar.xacro (robot description, xacro)
@@ -4,5 +4,5 @@
         <parent link="chassis"/>
         <child link="laser_frame"/>
-        <origin xyz="0.1 0 0.095" rpy="0 0 0"/>
+        <origin xyz="0.095 0 0.095" rpy="0 0 0"/>
     </joint>
     <link name="laser_frame">

File: robot_model_pkg/urdf/robot_core.xacro (robot description, xacro)
@@ -20,4 +20,12 @@
     <link name="base_link">
     </link>
+    <!-- BASE_FOOTPRINT LINK -->
+    <joint name="base_footprint_joint" type="fixed">
+        <parent link="base_link"/>
+        <child link="base_footprint"/>
+        <origin xyz="0 0 0" rpy="0 0 0"/>
+    </joint>
+    <link name="base_footprint">
+    </link>
     <!-- CHASSIS LINK -->
     <joint name="chassis_joint" type="fixed">
@@ -30,5 +38,5 @@
             <origin xyz="0.1 0 0.04"/>
             <geometry>
-                <box size="0.20 0.14 0.08"/>
+                <box size="0.220 0.14 0.08"/>
             </geometry>
             <material name="red"/>
