Commit message: Robot SLAM and Upstairs Map

File: robot_model_pkg/urdf/camera.xacro (robot description, xacro)
@@ -4,5 +4,5 @@
         <parent link="chassis"/>
         <child link="camera_link"/>
-        <origin xyz="0.205 0 0.07" rpy="0 0 0"/>
+        <origin xyz="0.225 0 0.07" rpy="0 0 0"/>
     </joint>
     <link name="camera_link">

Commit message: Camera and Depth Camera Added to Launch

File: robot_model_pkg/urdf/camera.xacro (robot description, xacro)
@@ -4,10 +4,10 @@
         <parent link="chassis"/>
         <child link="camera_link"/>
-        <origin xyz="0.225 0 0.07" rpy="0 0 0"/>
+        <origin xyz="0.215 0.019 0.099" rpy="0 0 0"/>
     </joint>
     <link name="camera_link">
         <visual>
             <geometry>
-                <box size=".01 .03 .03"/>
+                <box size=".01 .038 .038"/>
             </geometry>
             <material name="black"/>

File: robot_model_pkg/urdf/depth_camera.xacro (robot description, xacro)
@@ -4,10 +4,10 @@
         <parent link="chassis"/>
         <child link="depth_camera_link"/>
-        <origin xyz="0.205 0 0.07" rpy="0 0 0"/>
+        <origin xyz="0.195 -0.019 0.099" rpy="0 0 0"/>
     </joint>
     <link name="depth_camera_link">
         <visual>
             <geometry>
-                <box size=".01 .03 .03"/>
+                <box size=".01 .038 .038"/>
             </geometry>
             <material name="black"/>
@@ -39,5 +39,5 @@
             </camera>
             <plugin name="depth_camera_controller" filename="libgazebo_ros_camera.so">
-                <frame_name>camera_link_optical</frame_name>
+                <frame_name>depth_camera_link_optical</frame_name>
                 <mindepth>0.1</mindepth>
                 <maxdepth>100.0</maxdepth>

File: robot_model_pkg/urdf/robot.urdf.xacro (robot description, xacro)
@@ -12,4 +12,4 @@
     <xacro:include filename="lidar.xacro" />
     <xacro:include filename="camera.xacro" />
-    <!-- <xacro:include filename="depth_camera.xacro" /> -->
+    <xacro:include filename="depth_camera.xacro" />
 </robot>

Commit message: Updated URDF 5/3/25

File: robot_model_pkg/urdf/camera.xacro (robot description, xacro)
@@ -2,7 +2,7 @@
 <robot xmlns:xacro="http://www.ros.org/wiki/xacro" >
     <joint name="camera_joint" type="fixed">
-        <parent link="chassis"/>
+        <parent link="risers_link"/>
         <child link="camera_link"/>
-        <origin xyz="0.215 0.019 0.099" rpy="0 0 0"/>
+        <origin xyz="0.115 0.019 0.069" rpy="0 0 0"/>
     </joint>
     <link name="camera_link">
@@ -30,5 +30,5 @@
                 <image>
                     <format>R8G8B8</format>
-                    <width>640</width>
+                    <width>1280</width>
                     <height>480</height>
                 </image>

File: robot_model_pkg/urdf/depth_camera.xacro (robot description, xacro)
@@ -2,7 +2,7 @@
 <robot xmlns:xacro="http://www.ros.org/wiki/xacro" >
     <joint name="depth_camera_joint" type="fixed">
-        <parent link="chassis"/>
+        <parent link="risers_link"/>
         <child link="depth_camera_link"/>
-        <origin xyz="0.195 -0.019 0.099" rpy="0 0 0"/>
+        <origin xyz="0.115 -0.019 0.069" rpy="0 0 0"/>
     </joint>
     <link name="depth_camera_link">

File: robot_model_pkg/urdf/lidar.xacro (robot description, xacro)
@@ -2,7 +2,7 @@
 <robot xmlns:xacro="http://www.ros.org/wiki/xacro" >
     <joint name="laser_joint" type="fixed">
-        <parent link="chassis"/>
+        <parent link="risers_link"/>
         <child link="laser_frame"/>
-        <origin xyz="0.095 0 0.095" rpy="0 0 0"/>
+        <origin xyz="0.08 0 0.115" rpy="0 0 0"/>
     </joint>
     <link name="laser_frame">

File: robot_model_pkg/urdf/robot_core.xacro (robot description, xacro)
@@ -45,5 +45,5 @@
             <origin xyz="0.1 0 0.04"/>
             <geometry>
-                <box size="0.20 0.14 0.08"/>
+                <box size="0.220 0.14 0.08"/>
             </geometry>
         </collision>
@@ -53,4 +53,31 @@
     </link>
     <gazebo reference="chassis">
+        <material>Gazebo/Red</material>
+    </gazebo>
+    <!-- RISERS LINK   -->
+    <joint name="risers_joint" type="fixed">
+        <parent link="chassis"/>
+        <child link="risers_link"/>
+        <origin xyz="0.0 0 0.08"/>
+    </joint>
+    <link name="risers_link">
+        <visual>
+            <origin xyz="0.055 0 0.05"/>
+            <geometry>
+                <box size="0.110 0.12 0.1"/>
+            </geometry>
+            <material name="red"/>
+        </visual>
+        <collision>
+            <origin xyz="0.055 0 0.130"/>
+            <geometry>
+                <box size="0.110 0.12 0.1"/>
+            </geometry>
+        </collision>
+        <xacro:inertial_box mass=".1" x="0.110" y="0.12" z="0.05">
+            <origin xyz="0.055 0 0.130" rpy="0 0 0 "/>
+        </xacro:inertial_box>
+    </link>
+    <gazebo reference="risers_link">
         <material>Gazebo/Red</material>
     </gazebo>
