Commit message: Configured Gazebo launch.

File: robot_model_pkg/urdf/robot.urdf.xacro (robot description, xacro)
@@ -2,3 +2,5 @@
 <robot xmlns:xacro="http://www.ros.org/wiki/xacro" name="robot">
     <xacro:include filename="robot_core.xacro" />
+    <xacro:include filename="gazebo_control.xacro" />
+    <xacro:include filename="lidar.xacro" />
 </robot>

File: robot_model_pkg/urdf/robot_core.xacro (robot description, xacro)
@@ -1,4 +1,5 @@
 <?xml version="1.0"?>
 <robot xmlns:xacro="http://www.ros.org/wiki/xacro">
+    <xacro:include filename="inertial_macros.xacro"/>
     <material name="white">
         <color rgba="1 1 1 1"/>
@@ -33,10 +34,22 @@
             <material name="red"/>
         </visual>
+        <collision>
+            <origin xyz="0.1 0 0.04"/>
+            <geometry>
+                <box size="0.20 0.14 0.08"/>
+            </geometry>
+        </collision>
+        <xacro:inertial_box mass="1.7" x="0.20" y="0.14" z="0.08">
+            <origin xyz="0.1 0 0.04" rpy="0 0 0 "/>
+        </xacro:inertial_box>
     </link>
+    <gazebo reference="chassis">
+        <material>Gazebo/Red</material>
+    </gazebo>
     <!-- LEFT WHEEL LINK -->
     <joint name="left_wheel_joint" type="continuous">
         <parent link="base_link"/>
         <child link="left_wheel"/>
-        <origin xyz="0.0 0.1 0.0" rpy="-${pi/2} 0 0" />
+        <origin xyz="0.0 0.094 0.0" rpy="-${pi/2} 0 0" />
         <axis xyz="0 0 1"/>
     </joint>
@@ -48,10 +61,21 @@
             <material name="black"/>
         </visual>
+        <collision>
+            <geometry>
+                <cylinder radius="0.0215" length="0.035"/>
+            </geometry>
+        </collision>
+        <xacro:inertial_cylinder mass="0.1" length="0.035" radius="0.0215">
+            <origin xyz="0 0 0" rpy="0 0 0"/>
+        </xacro:inertial_cylinder>
     </link>
+    <gazebo reference="left_wheel">
+        <material>Gazebo/Black</material>
+    </gazebo>
     <!-- RIGHT WHEEL LINK -->
     <joint name="right_wheel_joint" type="continuous">
         <parent link="base_link"/>
         <child link="right_wheel"/>
-        <origin xyz="0.0 -0.1 0.0" rpy="${pi/2} 0 0" />
+        <origin xyz="0.0 -0.094 0.0" rpy="${pi/2} 0 0" />
         <axis xyz="0 0 -1"/>
     </joint>
@@ -63,4 +87,69 @@
             <material name="black"/>
         </visual>
+        <collision>
+            <geometry>
+                <cylinder radius="0.0215" length="0.035"/>
+            </geometry>
+        </collision>
+        <xacro:inertial_cylinder mass="0.1" length="0.035" radius="0.0215">
+            <origin xyz="0 0 0" rpy="0 0 0"/>
+        </xacro:inertial_cylinder>
     </link>
+    <gazebo reference="right_wheel">
+        <material>Gazebo/Black</material>
+    </gazebo>
+    <!-- FRONT CASTER WHEEL LINK -->
+    <joint name="front_caster_wheel_joint" type="fixed">
+        <parent link="chassis"/>
+        <child link="front_caster_wheel"/>
+        <origin xyz=".18 0.0 0.0"/>
+    </joint>
+    <link name="front_caster_wheel">
+        <visual>
+            <geometry>
+                <sphere radius="0.0215"/>
+            </geometry>
+            <material name="white"/>
+        </visual>
+        <collision>
+            <geometry>
+                <sphere radius="0.0215"/>
+            </geometry>
+        </collision>
+        <xacro:inertial_sphere mass="0.1" radius="0.0215">
+            <origin xyz="0 0 0" rpy="0 0 0"/>
+        </xacro:inertial_sphere>
+    </link>
+    <gazebo reference="front_caster_wheel">
+        <material>Gazebo/White</material>
+        <mu1 value=".001"/>
+        <mu2 value=".001"/>
+    </gazebo>
+    <!-- REAR CASTER WHEEL LINK -->
+    <joint name="rear_caster_wheel_joint" type="fixed">
+        <parent link="chassis"/>
+        <child link="rear_caster_wheel"/>
+        <origin xyz=".0215 0.0 0.0"/>
+    </joint>
+    <link name="rear_caster_wheel">
+        <visual>
+            <geometry>
+                <sphere radius="0.0215"/>
+            </geometry>
+            <material name="blue"/>
+        </visual>
+        <collision>
+            <geometry>
+                <sphere radius="0.0215"/>
+            </geometry>
+        </collision>
+        <xacro:inertial_sphere mass="0.1" radius="0.0215">
+            <origin xyz="0 0 0" rpy="0 0 0"/>
+        </xacro:inertial_sphere>
+    </link>
+    <gazebo reference="rear_caster_wheel">
+        <material>Gazebo/Blue</material>
+        <mu1 value=".001"/>
+        <mu2 value=".001"/>
+    </gazebo>
 </robot>

Commit message: Ros2 Control Updated

File: robot_model_pkg/urdf/robot.urdf.xacro (robot description, xacro)
@@ -1,7 +1,13 @@
 <?xml version="1.0"?>
 <robot xmlns:xacro="http://www.ros.org/wiki/xacro"  name="robot">
+    <xacro:arg name="use_ros2_control" default="true"/>
+    <xacro:arg name="sim_mode" default="false"/>
     <xacro:include filename="robot_core.xacro" />
-    <!-- <xacro:include filename="gazebo_control.xacro" /> -->
-    <xacro:include filename="ros2_control.xacro" />
+    <xacro:if value="$(arg use_ros2_control)">
+        <xacro:include filename="ros2_control.xacro" />
+    </xacro:if>
+    <xacro:unless value="$(arg use_ros2_control)">
+        <xacro:include filename="gazebo_control.xacro" />
+    </xacro:unless>
     <xacro:include filename="lidar.xacro" />
     <xacro:include filename="camera.xacro" />

File: robot_model_pkg/urdf/ros2_control.xacro (robot description, xacro)
@@ -1,61 +1,61 @@
 <?xml version="1.0"?>
 <robot xmlns:xacro="http://www.ros.org/wiki/xacro">
-    <ros2_control name="Robot" type="system">
-        <hardware>
-            <plugin>diffdrive_arduino/DiffDriveArduino</plugin>
-            <param name="left_wheel_name">left_wheel_joint</param>
-            <param name="right_wheel_name">right_wheel_joint</param>
-            <param name="loop_rate">30</param>
-            <param name="device">/dev/ttyUSB0</param>
-            <param name="baud_rate">57600</param>
-            <param name="timeout_ms">1000</param>
-            <param name="enc_counts_per_rev">3436</param>
-            <param name="pid_p">20</param>
-            <param name="pid_d">12</param>
-            <param name="pid_i">0</param>
-            <param name="pid_o">50</param>
-        </hardware>
-        <joint name="left_wheel_joint">
-            <command_interface name="velocity">
-                <param name="min">-10</param>
-                <param name="max">10</param>
-            </command_interface>
-            <state_interface name="velocity"/>
-            <state_interface name="position"/>
-        </joint>
-        <joint name="right_wheel_joint">
-            <command_interface name="velocity">
-                <param name="min">-10</param>
-                <param name="max">10</param>
-            </command_interface>
-            <state_interface name="velocity"/>
-            <state_interface name="position"/>
-        </joint>
-    </ros2_control>
- <!--  <ros2_control name="GazeboSystem" type="system">
-        <hardware>
-            <plugin>gazebo_ros2_control/GazeboSystem</plugin>
-        </hardware>
-        <joint name="left_wheel_joint">
-            <command_interface name="velocity">
-                <param name="min">-10</param>
-                <param name="max">10</param>
-            </command_interface>
-            <state_interface name="velocity"/>
-            <state_interface name="position"/>
-        </joint>
-        <joint name="right_wheel_joint">
-            <command_interface name="velocity">
-                <param name="min">-10</param>
-                <param name="max">10</param>
-            </command_interface>
-            <state_interface name="velocity"/>
-            <state_interface name="position"/>
-        </joint>
-    </ros2_control>
-    -->
+    <xacro:unless value="$(arg sim_mode)">
+        <ros2_control name="RealRobot" type="system">
+            <hardware>
+                <plugin>diffdrive_arduino/DiffDriveArduinoHardware</plugin>
+                <param name="left_wheel_name">left_wheel_joint</param>
+                <param name="right_wheel_name">right_wheel_joint</param>
+                <param name="loop_rate">30</param>
+                <param name="device">/dev/ttyUSB0</param>
+                <param name="baud_rate">57600</param>
+                <param name="timeout_ms">1000</param>
+                <param name="enc_counts_per_rev">3436</param>
+            </hardware>
+            <joint name="left_wheel_joint">
+                <command_interface name="velocity">
+                    <param name="min">-10</param>
+                    <param name="max">10</param>
+                </command_interface>
+                <state_interface name="position"/>
+                <state_interface name="velocity"/>
+            </joint>
+            <joint name="right_wheel_joint">
+                <command_interface name="velocity">
+                    <param name="min">-10</param>
+                    <param name="max">10</param>
+                </command_interface>
+                <state_interface name="position"/>
+                <state_interface name="velocity"/>
+            </joint>
+        </ros2_control>
+    </xacro:unless>
+    <xacro:if value="$(arg sim_mode)">
+        <ros2_control name="GazeboSystem" type="system">
+            <hardware>
+                <plugin>gazebo_ros2_control/GazeboSystem</plugin>
+            </hardware>
+            <joint name="left_wheel_joint">
+                <command_interface name="velocity">
+                    <param name="min">-10</param>
+                    <param name="max">10</param>
+                </command_interface>
+                <state_interface name="velocity"/>
+                <state_interface name="position"/>
+            </joint>
+            <joint name="right_wheel_joint">
+                <command_interface name="velocity">
+                    <param name="min">-10</param>
+                    <param name="max">10</param>
+                </command_interface>
+                <state_interface name="velocity"/>
+                <state_interface name="position"/>
+            </joint>
+        </ros2_control>
+    </xacro:if>
     <gazebo>
         <plugin name="gazebo_ros2_control" filename="libgazebo_ros2_control.so">
             <parameters>$(find robot_model_pkg)/config/my_controllers.yaml</parameters>
+            <parameters>$(find robot_model_pkg)/config/gaz_ros2_ctl_use_sim.yaml</parameters>
         </plugin>
     </gazebo>

Commit message: robot with arm controllers and nav2 working (turtlebot3 example)

File: robot_model_pkg/urdf/robot.urdf.xacro (robot description, xacro)
@@ -5,12 +5,14 @@
     <xacro:arg name="use_fake_hardware" default="false"/>
     <xacro:include filename="robot_core.xacro" />
-    <xacro:if value="$(arg use_ros2_control)">
-        <xacro:include filename="ros2_control.xacro" />
-    </xacro:if>
+    <xacro:include filename="robot_arm.xacro" />
+    <xacro:arm/>
     <xacro:include filename="lidar.xacro" />
     <xacro:include filename="camera.xacro" />
     <xacro:include filename="depth_camera.xacro" />
-    <xacro:include filename="robot_arm.xacro" />
-    <xacro:arm/>
+    <gazebo>
+        <plugin name="gazebo_ros2_control" filename="libgazebo_ros2_control.so">
+        <parameters>$(find robot_model_pkg)/config/gazebo_controller_manager.yaml</parameters>
+        </plugin>
+    </gazebo>
 </robot>
 <!--

File: robot_model_pkg/urdf/robot_arm.xacro (robot description, xacro)
@@ -310,4 +310,5 @@
     <axis xyz="0 -1 0"/>
     <limit effort="${prismatic_joint_effort}" lower="0.0" upper="${gripper_max_opening/2}" velocity="${prismatic_joint_velocity}"/>
+    <mimic joint="gripper_left_finger_joint" multiplier="1.0"/>
   </joint>
   <link name="gripper_right_finger">

File: robot_model_pkg/urdf/ros2_control.xacro (robot description, xacro)
@@ -54,9 +54,3 @@
         </ros2_control>
     </xacro:if>
-    <gazebo>
-        <plugin name="gazebo_ros2_control" filename="libgazebo_ros2_control.so">
-            <parameters>$(find robot_model_pkg)/config/my_controllers.yaml</parameters>
-            <parameters>$(find robot_model_pkg)/config/gaz_ros2_ctl_use_sim.yaml</parameters>
-        </plugin>
-    </gazebo>
 </robot>
