Commit message: arm pick and place working

File: arm/description/urdf/old2_r4bot_description.urdf.xacro (robot description, xacro)
@@ -12,13 +12,13 @@
   <xacro:property name="link1_width" value="0.1"/>
   <xacro:property name="link1_height" value="0.1"/>
-  <xacro:property name="link1_offset_y" value="0.08"/>
+  <xacro:property name="link1_offset_x" value="0.08"/>
   <xacro:property name="link1_offset_z" value="0.05"/>
   <xacro:property name="link1_mass" value="1.5"/>
   <!-- Link 2 Properties -->
-  <xacro:property name="link2_length" value="0.06"/>
+  <xacro:property name="link2_length" value="0.35"/>
   <xacro:property name="link2_width" value="0.06"/>
-  <xacro:property name="link2_height" value="0.35"/>
-  <xacro:property name="link2_offset_y" value="${link2_length/2}"/>
-  <xacro:property name="link2_offset_z" value="${link2_height/2}"/>
+  <xacro:property name="link2_height" value="0.06"/>
+  <xacro:property name="link2_offset_x" value="${link2_length/2}"/>
+  <xacro:property name="link2_offset_z" value="0.03"/>
   <xacro:property name="link2_mass" value="3.0"/>
   <!-- Link 3 Properties -->
@@ -27,5 +27,4 @@
   <xacro:property name="link3_height" value="0.06"/>
   <xacro:property name="link3_offset_x" value="${link3_length/2}"/>
-  <xacro:property name="link3_offset_y" value="${link3_width/2}"/>
   <xacro:property name="link3_offset_z" value="-0.03"/>
   <xacro:property name="link3_mass" value="2.0"/>
@@ -35,20 +34,19 @@
   <xacro:property name="link4_height" value="0.06"/>
   <xacro:property name="link4_offset_x" value="${link4_length/2}"/>
-  <xacro:property name="link4_offset_y" value="${link4_width/2}"/>
   <xacro:property name="link4_offset_z" value="0.03"/>
   <xacro:property name="link4_mass" value="1.0"/>
   <!-- Gripper Properties -->
-  <xacro:property name="gripper_base_length" value="0.02"/>
+  <xacro:property name="gripper_base_length" value="0.04"/>
   <xacro:property name="gripper_base_width" value="0.14"/>
-  <xacro:property name="gripper_base_height" value="0.04"/>
+  <xacro:property name="gripper_base_height" value="0.02"/>
   <xacro:property name="gripper_base_offset_z" value="0.03"/>
   <xacro:property name="gripper_base_mass" value="0.2"/>
-  <xacro:property name="gripper_finger_length" value="0.1"/>
+  <xacro:property name="gripper_finger_length" value="0.02"/>
   <xacro:property name="gripper_finger_width" value="0.02"/>
-  <xacro:property name="gripper_finger_height" value="0.02"/>
+  <xacro:property name="gripper_finger_height" value="0.1"/>
   <xacro:property name="gripper_finger_mass" value="0.1"/>
   <xacro:property name="gripper_max_opening" value="0.1"/>
   <!-- End Effector Properties -->
-  <xacro:property name="end_effector_offset_x" value="0.06"/>
+  <xacro:property name="end_effector_offset_z" value="0.06"/>
   <!-- ========== JOINT PROPERTIES ========== -->
   <!-- Joint angle variables (default values in radians) -->
@@ -73,9 +71,8 @@
   <!-- Joint origin offsets (calculated from link dimensions) -->
   <xacro:property name="joint_1_offset_z" value="${base_length}"/>
-  <xacro:property name="joint_2_offset_y" value="${link1_offset_y - link1_length/2}"/>
+  <xacro:property name="joint_2_offset_x" value="${link1_offset_x - link1_length/2}"/>
   <xacro:property name="joint_2_offset_z" value="${link1_offset_z}"/>
-  <xacro:property name="joint_3_offset_z" value="${link2_height}"/>
+  <xacro:property name="joint_3_offset_x" value="${link2_length}"/>
   <xacro:property name="joint_4_offset_x" value="${link3_length}"/>
-  <xacro:property name="joint_4_offset_y" value="${link4_offset_y}"/>
   <xacro:property name="gripper_base_joint_offset_x" value="${link4_offset_x + link4_length/2}"/>
   <!-- ========== COLOR PROPERTIES ========== -->
@@ -132,5 +129,5 @@
     <parent link="base_link"/>
     <child link="link_1"/>
-    <origin xyz="0 0 ${joint_1_offset_z}" rpy="0 0 0"/>
+    <origin xyz="0 0 ${joint_1_offset_z}" rpy="0 0 ${joint_1_angle}"/>
     <axis xyz="0 0 1"/>
     <limit effort="${revolute_joint_effort}" lower="${joint_1_lower_limit}" upper="${joint_1_upper_limit}" velocity="${revolute_joint_velocity}"/>
@@ -138,5 +135,5 @@
   <link name="link_1">
     <visual>
-      <origin xyz="0 ${-link1_offset_y} ${link1_offset_z}" rpy="0 0 0"/>
+      <origin xyz="${link1_offset_x} 0 ${link1_offset_z}" rpy="0 0 0"/>
       <geometry>
         <box size="${link1_length} ${link1_width} ${link1_height}"/>
@@ -147,5 +144,5 @@
     </visual>
     <collision>
-      <origin xyz="0 ${-link1_offset_y} ${link1_offset_z}" rpy="0 0 0"/>
+      <origin xyz="${link1_offset_x} 0 ${link1_offset_z}" rpy="0 0 0"/>
       <geometry>
         <box size="${link1_length} ${link1_width} ${link1_height}"/>
@@ -161,11 +158,11 @@
     <parent link="link_1"/>
     <child link="link_2"/>
-    <origin xyz="0 ${-joint_2_offset_y} ${joint_2_offset_z}" rpy="0 0 0"/>
-    <axis xyz="0 1 0"/>
+    <origin xyz="${joint_2_offset_x} 0 ${joint_2_offset_z}" rpy="0 ${-pi/2} ${joint_2_angle}"/>
+    <axis xyz="0 0 1"/>
     <limit effort="${revolute_joint_effort}" lower="${joint_2_lower_limit}" upper="${joint_2_upper_limit}" velocity="${revolute_joint_velocity}"/>
   </joint>
   <link name="link_2">
     <visual>
-      <origin xyz="0 ${link2_offset_y} ${link2_offset_z}" rpy="0 0 0"/>
+      <origin xyz="${link2_offset_x} 0 ${link2_offset_z}" rpy="0 0 0"/>
       <geometry>
         <box size="${link2_length} ${link2_width} ${link2_height}"/>
@@ -176,5 +173,5 @@
     </visual>
     <collision>
-      <origin xyz="0 ${link2_offset_y} ${link2_offset_z}" rpy="0 0 0"/>
+      <origin xyz="${link2_offset_x} 0 ${link2_offset_z}" rpy="0 0 0"/>
       <geometry>
         <box size="${link2_length} ${link2_width} ${link2_height}"/>
@@ -190,11 +187,11 @@
     <parent link="link_2"/>
     <child link="link_3"/>
-    <origin xyz="0 0 ${joint_3_offset_z}" rpy="0 0 0"/>
-    <axis xyz="0 1 0"/>
+    <origin xyz="${joint_3_offset_x} 0 0" rpy="0 0 ${joint_3_angle}"/>
+    <axis xyz="0 0 1"/>
     <limit effort="${revolute_joint_effort}" lower="${joint_3_lower_limit}" upper="${joint_3_upper_limit}" velocity="${revolute_joint_velocity}"/>
   </joint>
   <link name="link_3">
     <visual>
-      <origin xyz="${link3_offset_x} ${-link3_offset_y} 0" rpy="0 0 0"/>
+      <origin xyz="${link3_offset_x} 0 ${link3_offset_z}" rpy="0 0 0"/>
       <geometry>
         <box size="${link3_length} ${link3_width} ${link3_height}"/>
@@ -205,5 +202,5 @@
     </visual>
     <collision>
-      <origin xyz="${link3_offset_x} ${-link3_offset_y} 0" rpy="0 0 0"/>
+      <origin xyz="${link3_offset_x} 0 ${link3_offset_z}" rpy="0 0 0"/>
       <geometry>
         <box size="${link3_length} ${link3_width} ${link3_height}"/>
@@ -219,11 +216,11 @@
     <parent link="link_3"/>
     <child link="link_4"/>
-    <origin xyz="${joint_4_offset_x} 0 0" rpy="0 0 0"/>
-    <axis xyz="0 1 0"/>
+    <origin xyz="${joint_4_offset_x} 0 0" rpy="0 0 ${joint_4_angle}"/>
+    <axis xyz="0 0 1"/>
     <limit effort="${revolute_joint_effort}" lower="${joint_4_lower_limit}" upper="${joint_4_upper_limit}" velocity="${revolute_joint_velocity}"/>
   </joint>
   <link name="link_4">
     <visual>
-      <origin xyz="${link4_offset_x} ${link4_offset_y} 0" rpy="0 0 0"/>
+      <origin xyz="${link4_offset_x} 0 ${link4_offset_z}" rpy="0 0 0"/>
       <geometry>
         <box size="${link4_length} ${link4_width} ${link4_height}"/>
@@ -234,5 +231,5 @@
     </visual>
     <collision>
-      <origin xyz="${link4_offset_x} 0 0" rpy="0 0 0"/>
+      <origin xyz="${link4_offset_x} 0 ${link4_offset_z}" rpy="0 0 0"/>
       <geometry>
         <box size="${link4_length} ${link4_width} ${link4_height}"/>
@@ -249,5 +246,5 @@
     <parent link="link_4"/>
     <child link="gripper_base"/>
-    <origin xyz="${link4_length} ${link4_offset_y} 0" rpy="0 0 0"/>
+    <origin xyz="${link4_length} 0 ${link4_height/2}" rpy="${pi/2} ${pi} ${pi/2}"/>
   </joint>
   <link name="gripper_base">
@@ -277,11 +274,11 @@
     <parent link="gripper_base"/>
     <child link="gripper_left_finger"/>
-    <origin xyz="0 0 0" rpy="0 0 0"/>
-    <axis xyz="0 1 0"/>
+    <origin xyz="0 -0.005 ${gripper_base_height/2}" rpy="0 0 0"/>
+    <axis xyz="0 -1 0"/>
     <limit effort="${prismatic_joint_effort}" lower="0.0" upper="${gripper_max_opening/2}" velocity="${prismatic_joint_velocity}"/>
   </joint>
   <link name="gripper_left_finger">
     <visual>
-      <origin xyz="${gripper_finger_length/2} ${gripper_finger_width/2} 0" rpy="0 0 0"/>
+      <origin xyz="0 ${-gripper_finger_width/2} ${gripper_finger_height/2}" rpy="0 0 0"/>
       <geometry>
         <box size="${gripper_finger_length} ${gripper_finger_width} ${gripper_finger_height}"/>
@@ -292,5 +289,5 @@
     </visual>
     <collision>
-      <origin xyz="${gripper_finger_length/2} ${gripper_finger_width/2} 0" rpy="0 0 0"/>
+      <origin xyz="0 ${-gripper_finger_width/2} ${gripper_finger_height/2}" rpy="0 0 0"/>
       <geometry>
         <box size="${gripper_finger_length} ${gripper_finger_width} ${gripper_finger_height}"/>
@@ -307,11 +304,11 @@
     <parent link="gripper_base"/>
     <child link="gripper_right_finger"/>
-    <origin xyz="0 0 0" rpy="0 0 0"/>
-    <axis xyz="0 -1 0"/>
+    <origin xyz="0 0.005 ${gripper_base_height/2}" rpy="0 0 0"/>
+    <axis xyz="0 1 0"/>
     <limit effort="${prismatic_joint_effort}" lower="0.0" upper="${gripper_max_opening/2}" velocity="${prismatic_joint_velocity}"/>
   </joint>
   <link name="gripper_right_finger">
     <visual>
-      <origin xyz="${gripper_finger_length/2} ${-gripper_finger_width/2} 0" rpy="0 0 0"/>
+      <origin xyz="0 ${gripper_finger_width/2} ${gripper_finger_height/2}" rpy="0 0 0"/>
       <geometry>
         <box size="${gripper_finger_length} ${gripper_finger_width} ${gripper_finger_height}"/>
@@ -322,5 +319,5 @@
     </visual>
     <collision>
-      <origin xyz="${gripper_finger_length/2} ${-gripper_finger_width/2} 0" rpy="0 0 0"/>
+      <origin xyz="0 ${gripper_finger_width/2} ${gripper_finger_height/2}" rpy="0 0 0"/>
       <geometry>
         <box size="${gripper_finger_length} ${gripper_finger_width} ${gripper_finger_height}"/>
@@ -337,5 +334,5 @@
     <parent link="gripper_base"/>
     <child link="end_effector_roll_virtual"/>
-    <origin xyz="${end_effector_offset_x} 0 0" rpy="0 0 0"/>
+    <origin xyz="0 0 ${end_effector_offset_z}" rpy="0 0 0"/>
     <axis xyz="0 0 1"/>
     <limit effort="0.0" lower="-3.14" upper="3.14" velocity="0.0"/>

File: arm/description/urdf/old_r4bot_description.urdf.xacro (robot description, xacro)
@@ -12,13 +12,13 @@
   <xacro:property name="link1_width" value="0.1"/>
   <xacro:property name="link1_height" value="0.1"/>
-  <xacro:property name="link1_offset_y" value="0.08"/>
+  <xacro:property name="link1_offset_x" value="0.08"/>
   <xacro:property name="link1_offset_z" value="0.05"/>
   <xacro:property name="link1_mass" value="1.5"/>
   <!-- Link 2 Properties -->
-  <xacro:property name="link2_length" value="0.06"/>
+  <xacro:property name="link2_length" value="0.35"/>
   <xacro:property name="link2_width" value="0.06"/>
-  <xacro:property name="link2_height" value="0.35"/>
-  <xacro:property name="link2_offset_y" value="${link2_length/2}"/>
-  <xacro:property name="link2_offset_z" value="${link2_height/2}"/>
+  <xacro:property name="link2_height" value="0.06"/>
+  <xacro:property name="link2_offset_x" value="${link2_length/2}"/>
+  <xacro:property name="link2_offset_z" value="0.03"/>
   <xacro:property name="link2_mass" value="3.0"/>
   <!-- Link 3 Properties -->
@@ -27,5 +27,4 @@
   <xacro:property name="link3_height" value="0.06"/>
   <xacro:property name="link3_offset_x" value="${link3_length/2}"/>
-  <xacro:property name="link3_offset_y" value="${link3_width/2}"/>
   <xacro:property name="link3_offset_z" value="-0.03"/>
   <xacro:property name="link3_mass" value="2.0"/>
@@ -35,11 +34,10 @@
   <xacro:property name="link4_height" value="0.06"/>
   <xacro:property name="link4_offset_x" value="${link4_length/2}"/>
-  <xacro:property name="link4_offset_y" value="${link4_width/2}"/>
   <xacro:property name="link4_offset_z" value="0.03"/>
   <xacro:property name="link4_mass" value="1.0"/>
   <!-- Gripper Properties -->
   <xacro:property name="gripper_base_length" value="0.02"/>
-  <xacro:property name="gripper_base_width" value="0.14"/>
-  <xacro:property name="gripper_base_height" value="0.04"/>
+  <xacro:property name="gripper_base_width" value="0.04"/>
+  <xacro:property name="gripper_base_height" value="0.12"/>
   <xacro:property name="gripper_base_offset_z" value="0.03"/>
   <xacro:property name="gripper_base_mass" value="0.2"/>
@@ -50,5 +48,5 @@
   <xacro:property name="gripper_max_opening" value="0.1"/>
   <!-- End Effector Properties -->
-  <xacro:property name="end_effector_offset_x" value="0.06"/>
+  <xacro:property name="end_effector_offset_x" value="0.04"/>
   <!-- ========== JOINT PROPERTIES ========== -->
   <!-- Joint angle variables (default values in radians) -->
@@ -73,9 +71,8 @@
   <!-- Joint origin offsets (calculated from link dimensions) -->
   <xacro:property name="joint_1_offset_z" value="${base_length}"/>
-  <xacro:property name="joint_2_offset_y" value="${link1_offset_y - link1_length/2}"/>
+  <xacro:property name="joint_2_offset_x" value="${link1_offset_x - link1_length/2}"/>
   <xacro:property name="joint_2_offset_z" value="${link1_offset_z}"/>
-  <xacro:property name="joint_3_offset_z" value="${link2_height}"/>
+  <xacro:property name="joint_3_offset_x" value="${link2_length}"/>
   <xacro:property name="joint_4_offset_x" value="${link3_length}"/>
-  <xacro:property name="joint_4_offset_y" value="${link4_offset_y}"/>
   <xacro:property name="gripper_base_joint_offset_x" value="${link4_offset_x + link4_length/2}"/>
   <!-- ========== COLOR PROPERTIES ========== -->
@@ -132,5 +129,5 @@
     <parent link="base_link"/>
     <child link="link_1"/>
-    <origin xyz="0 0 ${joint_1_offset_z}" rpy="0 0 0"/>
+    <origin xyz="0 0 ${joint_1_offset_z}" rpy="0 0 ${joint_1_angle}"/>
     <axis xyz="0 0 1"/>
     <limit effort="${revolute_joint_effort}" lower="${joint_1_lower_limit}" upper="${joint_1_upper_limit}" velocity="${revolute_joint_velocity}"/>
@@ -138,5 +135,5 @@
   <link name="link_1">
     <visual>
-      <origin xyz="0 ${-link1_offset_y} ${link1_offset_z}" rpy="0 0 0"/>
+      <origin xyz="${link1_offset_x} 0 ${link1_offset_z}" rpy="0 0 0"/>
       <geometry>
         <box size="${link1_length} ${link1_width} ${link1_height}"/>
@@ -147,5 +144,5 @@
     </visual>
     <collision>
-      <origin xyz="0 ${-link1_offset_y} ${link1_offset_z}" rpy="0 0 0"/>
+      <origin xyz="${link1_offset_x} 0 ${link1_offset_z}" rpy="0 0 0"/>
       <geometry>
         <box size="${link1_length} ${link1_width} ${link1_height}"/>
@@ -161,11 +158,11 @@
     <parent link="link_1"/>
     <child link="link_2"/>
-    <origin xyz="0 ${-joint_2_offset_y} ${joint_2_offset_z}" rpy="0 0 0"/>
-    <axis xyz="0 1 0"/>
+    <origin xyz="${joint_2_offset_x} 0 ${joint_2_offset_z}" rpy="0 ${-pi/2} ${joint_2_angle}"/>
+    <axis xyz="0 0 1"/>
     <limit effort="${revolute_joint_effort}" lower="${joint_2_lower_limit}" upper="${joint_2_upper_limit}" velocity="${revolute_joint_velocity}"/>
   </joint>
   <link name="link_2">
     <visual>
-      <origin xyz="0 ${link2_offset_y} ${link2_offset_z}" rpy="0 0 0"/>
+      <origin xyz="${link2_offset_x} 0 ${link2_offset_z}" rpy="0 0 0"/>
       <geometry>
         <box size="${link2_length} ${link2_width} ${link2_height}"/>
@@ -176,5 +173,5 @@
     </visual>
     <collision>
-      <origin xyz="0 ${link2_offset_y} ${link2_offset_z}" rpy="0 0 0"/>
+      <origin xyz="${link2_offset_x} 0 ${link2_offset_z}" rpy="0 0 0"/>
       <geometry>
         <box size="${link2_length} ${link2_width} ${link2_height}"/>
@@ -190,11 +187,11 @@
     <parent link="link_2"/>
     <child link="link_3"/>
-    <origin xyz="0 0 ${joint_3_offset_z}" rpy="0 0 0"/>
-    <axis xyz="0 1 0"/>
+    <origin xyz="${joint_3_offset_x} 0 0" rpy="0 0 ${joint_3_angle}"/>
+    <axis xyz="0 0 1"/>
     <limit effort="${revolute_joint_effort}" lower="${joint_3_lower_limit}" upper="${joint_3_upper_limit}" velocity="${revolute_joint_velocity}"/>
   </joint>
   <link name="link_3">
     <visual>
-      <origin xyz="${link3_offset_x} ${-link3_offset_y} 0" rpy="0 0 0"/>
+      <origin xyz="${link3_offset_x} 0 ${link3_offset_z}" rpy="0 0 0"/>
       <geometry>
         <box size="${link3_length} ${link3_width} ${link3_height}"/>
@@ -205,5 +202,5 @@
     </visual>
     <collision>
-      <origin xyz="${link3_offset_x} ${-link3_offset_y} 0" rpy="0 0 0"/>
+      <origin xyz="${link3_offset_x} 0 ${link3_offset_z}" rpy="0 0 0"/>
       <geometry>
         <box size="${link3_length} ${link3_width} ${link3_height}"/>
@@ -219,11 +216,11 @@
     <parent link="link_3"/>
     <child link="link_4"/>
-    <origin xyz="${joint_4_offset_x} 0 0" rpy="0 0 0"/>
-    <axis xyz="0 1 0"/>
+    <origin xyz="${joint_4_offset_x} 0 0" rpy="0 0 ${joint_4_angle}"/>
+    <axis xyz="0 0 1"/>
     <limit effort="${revolute_joint_effort}" lower="${joint_4_lower_limit}" upper="${joint_4_upper_limit}" velocity="${revolute_joint_velocity}"/>
   </joint>
   <link name="link_4">
     <visual>
-      <origin xyz="${link4_offset_x} ${link4_offset_y} 0" rpy="0 0 0"/>
+      <origin xyz="${link4_offset_x} 0 ${link4_offset_z}" rpy="0 0 0"/>
       <geometry>
         <box size="${link4_length} ${link4_width} ${link4_height}"/>
@@ -234,5 +231,5 @@
     </visual>
     <collision>
-      <origin xyz="${link4_offset_x} 0 0" rpy="0 0 0"/>
+      <origin xyz="${link4_offset_x} 0 ${link4_offset_z}" rpy="0 0 0"/>
       <geometry>
         <box size="${link4_length} ${link4_width} ${link4_height}"/>
@@ -249,5 +246,5 @@
     <parent link="link_4"/>
     <child link="gripper_base"/>
-    <origin xyz="${link4_length} ${link4_offset_y} 0" rpy="0 0 0"/>
+    <origin xyz="${gripper_base_joint_offset_x} 0 ${gripper_base_offset_z}" rpy="0 0 0"/>
   </joint>
   <link name="gripper_base">
@@ -277,11 +274,11 @@
     <parent link="gripper_base"/>
     <child link="gripper_left_finger"/>
-    <origin xyz="0 0 0" rpy="0 0 0"/>
-    <axis xyz="0 1 0"/>
+    <origin xyz="0 0 ${gripper_finger_height/2}" rpy="0 0 0"/>
+    <axis xyz="0 0 1"/>
     <limit effort="${prismatic_joint_effort}" lower="0.0" upper="${gripper_max_opening/2}" velocity="${prismatic_joint_velocity}"/>
   </joint>
   <link name="gripper_left_finger">
     <visual>
-      <origin xyz="${gripper_finger_length/2} ${gripper_finger_width/2} 0" rpy="0 0 0"/>
+      <origin xyz="${gripper_finger_length/2} 0 0" rpy="0 0 0"/>
       <geometry>
         <box size="${gripper_finger_length} ${gripper_finger_width} ${gripper_finger_height}"/>
@@ -292,5 +289,5 @@
     </visual>
     <collision>
-      <origin xyz="${gripper_finger_length/2} ${gripper_finger_width/2} 0" rpy="0 0 0"/>
+      <origin xyz="${gripper_finger_length/2} 0 0" rpy="0 0 0"/>
       <geometry>
         <box size="${gripper_finger_length} ${gripper_finger_width} ${gripper_finger_height}"/>
@@ -299,5 +296,5 @@
     <inertial>
       <mass value="${gripper_finger_mass}"/>
-      <origin xyz="0 ${-gripper_finger_width/2} ${gripper_finger_height/2}" rpy="0 0 0"/>
+      <origin xyz="${gripper_finger_length/2} 0 0" rpy="0 0 0"/>
       <inertia ixx="0.00005" ixy="0.0" ixz="0.0" iyy="0.00005" iyz="0.0" izz="0.00005"/>
     </inertial>
@@ -307,11 +304,12 @@
     <parent link="gripper_base"/>
     <child link="gripper_right_finger"/>
-    <origin xyz="0 0 0" rpy="0 0 0"/>
-    <axis xyz="0 -1 0"/>
+    <origin xyz="0 0 ${-gripper_finger_height/2}" rpy="0 0 0"/>
+    <axis xyz="0 0 -1"/>
     <limit effort="${prismatic_joint_effort}" lower="0.0" upper="${gripper_max_opening/2}" velocity="${prismatic_joint_velocity}"/>
+    <mimic joint="gripper_left_finger_joint" multiplier="1.0" offset="0.0"/>
   </joint>
   <link name="gripper_right_finger">
     <visual>
-      <origin xyz="${gripper_finger_length/2} ${-gripper_finger_width/2} 0" rpy="0 0 0"/>
+      <origin xyz="${gripper_finger_length/2} 0 0" rpy="0 0 0"/>
       <geometry>
         <box size="${gripper_finger_length} ${gripper_finger_width} ${gripper_finger_height}"/>
@@ -322,5 +320,5 @@
     </visual>
     <collision>
-      <origin xyz="${gripper_finger_length/2} ${-gripper_finger_width/2} 0" rpy="0 0 0"/>
+      <origin xyz="${gripper_finger_length/2} 0 0" rpy="0 0 0"/>
       <geometry>
         <box size="${gripper_finger_length} ${gripper_finger_width} ${gripper_finger_height}"/>
@@ -329,34 +327,16 @@
     <inertial>
       <mass value="${gripper_finger_mass}"/>
-      <origin xyz="0 ${gripper_finger_width/2} ${gripper_finger_height/2}" rpy="0 0 0"/>
+      <origin xyz="${gripper_finger_length/2} 0 0" rpy="0 0 0"/>
       <inertia ixx="0.00005" ixy="0.0" ixz="0.0" iyy="0.00005" iyz="0.0" izz="0.00005"/>
     </inertial>
   </link>
   <!-- End effector frame (for convenience in motion planning) -->
-  <joint name="end_effector_roll_virtual_joint" type="revolute">
+  <joint name="end_effector_joint" type="fixed">
     <parent link="gripper_base"/>
-    <child link="end_effector_roll_virtual"/>
+    <child link="end_effector"/>
     <origin xyz="${end_effector_offset_x} 0 0" rpy="0 0 0"/>
-    <axis xyz="0 0 1"/>
-    <limit effort="0.0" lower="-3.14" upper="3.14" velocity="0.0"/>
-  </joint>
-  <link name="end_effector_roll_virtual">
-  </link>
-  <joint name="end_effector_yaw_virtual_joint" type="revolute">
-    <parent link="end_effector_roll_virtual"/>
-    <child link="end_effector_yaw_virtual"/>
-    <origin xyz="0 0 0" rpy="0 0 0"/>
-    <axis xyz="0 0 1"/>
-    <limit effort="0.0" lower="-3.14" upper="3.14" velocity="0.0"/>
-  </joint>
-  <link name="end_effector_yaw_virtual">
-  </link>
-  <!-- End effector frame -->
-  <joint name="end_effector_joint" type="fixed">
-    <parent link="end_effector_yaw_virtual"/>
-    <child link="end_effector_frame"/>
-    <origin xyz="0 0 0" rpy="0 0 0"/>
-  </joint>
-  <link name="end_effector_frame">
+  </joint>
+  <link name="end_effector">
+    <!-- This is a virtual link for end effector positioning -->
   </link>
   </xacro:macro>
