Commit message: arm pick and place working

File: arm/description/urdf/r4bot.ros2_control.xacro (robot description, xacro)
@@ -8,6 +8,6 @@
       <joint name="joint_1">
         <command_interface name="position">
-          <param name="min">${-pi}</param>
-          <param name="max">${pi}</param>
+          <param name="min">${-pi/2}</param>
+          <param name="max">${pi/2}</param>
         </command_interface>
         <state_interface name="position">
@@ -18,6 +18,6 @@
       <joint name="joint_2">
         <command_interface name="position">
-          <param name="min">${pi}</param>
-          <param name="max">${pi}</param>
+          <param name="min">${-pi/2}</param>
+          <param name="max">${pi/2}</param>
         </command_interface>
         <state_interface name="position">
@@ -28,6 +28,6 @@
       <joint name="joint_3">
         <command_interface name="position">
-          <param name="min">${-pi}</param>
-          <param name="max">${pi}</param>
+          <param name="min">${-pi/2}</param>
+          <param name="max">${pi/2}</param>
         </command_interface>
         <state_interface name="position">
@@ -38,6 +38,6 @@
       <joint name="joint_4">
         <command_interface name="position">
-          <param name="min">${-pi}</param>
-          <param name="max">${pi}</param>
+          <param name="min">${-pi/2}</param>
+          <param name="max">${pi/2}</param>
         </command_interface>
         <state_interface name="position">

File: arm/description/urdf/r4bot.urdf.xacro (robot description, xacro)
@@ -1,4 +1,4 @@
 <?xml version="1.0"?>
-<robot xmlns:xacro="http://wiki.ros.org/xacro" name="r6bot">
+<robot xmlns:xacro="http://wiki.ros.org/xacro" name="r4bot">
   <!-- Import r6bot macro -->
   <xacro:include filename="$(find arm)/description/urdf/r4bot_description.urdf.xacro"/>
@@ -6,5 +6,5 @@
   <link name="world"/>
   <xacro:arm/>
-  <!-- Import r6bot ros2_control description -->
+  <!-- Import r4bot ros2_control description -->
   <xacro:include filename="$(find arm)/description/urdf/r4bot.ros2_control.xacro" />
   <xacro:r4bot_ros2_control name="r4bot"/>

File: arm_moveit_config/config/r4bot.ros2_control.xacro (robot description, xacro)
@@ -1,5 +1,5 @@
 <?xml version="1.0"?>
 <robot xmlns:xacro="http://www.ros.org/wiki/xacro">
-    <xacro:macro name="r6bot_ros2_control" params="name initial_positions_file">
+    <xacro:macro name="r4bot_ros2_control" params="name initial_positions_file">
         <xacro:property name="initial_positions" value="${load_yaml(initial_positions_file)['initial_positions']}"/>
         <ros2_control name="${name}" type="system">
@@ -36,4 +36,18 @@
                 <state_interface name="velocity"/>
             </joint>
+            <joint name="end_effector_roll_virtual_joint">
+                <command_interface name="position"/>
+                <state_interface name="position">
+                  <param name="initial_value">${initial_positions['end_effector_roll_virtual_joint']}</param>
+                </state_interface>
+                <state_interface name="velocity"/>
+            </joint>
+            <joint name="end_effector_yaw_virtual_joint">
+                <command_interface name="position"/>
+                <state_interface name="position">
+                  <param name="initial_value">${initial_positions['end_effector_yaw_virtual_joint']}</param>
+                </state_interface>
+                <state_interface name="velocity"/>
+            </joint>
             <joint name="gripper_left_finger_joint">
                 <command_interface name="position"/>
@@ -43,4 +57,11 @@
                 <state_interface name="velocity"/>
             </joint>
+            <joint name="gripper_right_finger_joint">
+                <command_interface name="position"/>
+                <state_interface name="position">
+                  <param name="initial_value">${initial_positions['gripper_right_finger_joint']}</param>
+                </state_interface>
+                <state_interface name="velocity"/>
+            </joint>
         </ros2_control>
     </xacro:macro>
