Commit message: Arm added to robot in rviz and gazebo sim, controllers properly configure. Config built, but controllers not configuring.

File: arm/description/urdf/r4bot.ros2_control.xacro (robot description, xacro)
@@ -54,4 +54,24 @@
         <state_interface name="torque.z"/>
       </sensor>
+      <joint name="gripper_left_finger_joint">
+        <command_interface name="position">
+          <param name="min">0.0</param>
+          <param name="max">0.05</param>
+        </command_interface>
+        <state_interface name="position">
+          <param name="initial_value">0.0</param>
+        </state_interface>
+        <state_interface name="velocity"/>
+      </joint>
+      <joint name="gripper_right_finger_joint">
+        <command_interface name="position">
+          <param name="min">0.0</param>
+          <param name="max">0.05</param>
+        </command_interface>
+        <state_interface name="position">
+          <param name="initial_value">0.0</param>
+        </state_interface>
+        <state_interface name="velocity"/>
+      </joint>
     </ros2_control>
   </xacro:macro>

File: robot_model_pkg/urdf/camera.xacro (robot description, xacro)
@@ -4,5 +4,5 @@
         <parent link="risers_link"/>
         <child link="camera_link"/>
-        <origin xyz="0.115 0.019 0.069" rpy="0 0 0"/>
+        <origin xyz="0.115 -0.019 0.069" rpy="0 0 0"/>
     </joint>
     <link name="camera_link">

File: robot_model_pkg/urdf/depth_camera.xacro (robot description, xacro)
@@ -4,5 +4,5 @@
         <parent link="risers_link"/>
         <child link="depth_camera_link"/>
-        <origin xyz="0.115 -0.019 0.069" rpy="0 0 0"/>
+        <origin xyz="0.115 0.019 0.069" rpy="0 0 0"/>
     </joint>
     <link name="depth_camera_link">
