Commit message: Nav2 and Moveit Working in Gazebo

File: robot_arm/ros2_control/base_arm_system.ros2_control.xacro (robot description, xacro)
@@ -6,5 +6,5 @@
 -->
 <robot xmlns:xacro="http://www.ros.org/wiki/xacro">
-  <xacro:macro name="base_arm_system" params="name prefix use_sim:=^|false use_fake_hardware:=^|false fake_sensor_commands:=^|false">
+  <xacro:macro name="base_arm_system" params="name prefix use_sim_time:=^|false use_fake_hardware:=^|false fake_sensor_commands:=^|false">
     <ros2_control name="${name}" type="system">
       <hardware>
@@ -117,6 +117,4 @@
       </joint>
       <joint name="gripper_right_finger_joint">
-        <param name="mimic">gripper_left_finger_joint</param>
-        <param name="multiplier">1</param>
         <command_interface name="position">
           <param name="min">-0</param>
@@ -130,4 +128,30 @@
         </state_interface>
       </joint>
+      <!--
+      <joint name="end_effector_roll_joint">
+        <command_interface name="position">
+          <param name="min">-3.14</param>
+          <param name="max">3.14</param>
+        </command_interface>
+        <state_interface name="position">
+          <param name="initial_value">0.0</param>
+        </state_interface>
+        <state_interface name="velocity">
+          <param name="initial_value">0.0</param>
+        </state_interface>
+      </joint>
+      <joint name="end_effector_yaw_joint">
+        <command_interface name="position">
+          <param name="min">-3.14</param>
+          <param name="max">3.14</param>
+        </command_interface>
+        <state_interface name="position">
+          <param name="initial_value">0.0</param>
+        </state_interface>
+        <state_interface name="velocity">
+          <param name="initial_value">0.0</param>
+        </state_interface>
+      </joint>
+    -->
     </ros2_control>
   </xacro:macro>

File: robot_arm/urdf/camera.xacro (robot description, xacro)
@@ -4,5 +4,5 @@
         <parent link="risers_link"/>
         <child link="camera_link"/>
-        <origin xyz="0.115 -0.019 0.069" rpy="0 0 0"/>
+        <origin xyz="0.115 0 0.069" rpy="0 0 0"/>
     </joint>
     <link name="camera_link">

File: robot_arm/urdf/depth_camera.xacro (robot description, xacro)
@@ -4,5 +4,5 @@
         <parent link="risers_link"/>
         <child link="depth_camera_link"/>
-        <origin xyz="0.115 0.019 0.069" rpy="0 0 0"/>
+        <origin xyz="0.115 0.038 0.069" rpy="0 0 0"/>
     </joint>
     <link name="depth_camera_link">

File: robot_arm/urdf/robot_arm.xacro (robot description, xacro)
@@ -310,5 +310,4 @@
     <axis xyz="0 -1 0"/>
     <limit effort="${prismatic_joint_effort}" lower="0.0" upper="${gripper_max_opening/2}" velocity="${prismatic_joint_velocity}"/>
-    <mimic joint="gripper_left_finger_joint" multiplier="1" offset="0"/>
   </joint>
   <link name="gripper_right_finger">
@@ -335,29 +334,60 @@
   </link>
   <!-- End effector frame (for convenience in motion planning) -->
-  <joint name="end_effector_roll_virtual_joint" type="revolute">
+  <joint name="end_effector_roll_joint" type="fixed">
     <parent link="gripper_base"/>
-    <child link="end_effector_roll_virtual"/>
+    <child link="end_effector_roll"/>
     <origin xyz="${end_effector_offset_x} 0 0" rpy="0 0 0"/>
+    <!--
+    <axis xyz="1 0 0"/>
+    <limit effort="0.0" lower="-3.14" upper="3.14" velocity="1"/>
+  -->
+  </joint>
+  <link name="end_effector_roll">
+    <visual>
+      <origin xyz="0 0 0" rpy="0 0 0"/>
+      <geometry>
+        <box size="0.01 0.01 0.01"/>
+      </geometry>
+      <material name="end_effector_roll_material">
+        <color rgba="${green}"/>
+      </material>
+    </visual>
+  </link>
+  <joint name="end_effector_yaw_joint" type="fixed">
+    <parent link="end_effector_roll"/>
+    <child link="end_effector_yaw"/>
+    <origin xyz="0 0 0" rpy="0 0 0"/>
+    <!--
     <axis xyz="0 0 1"/>
-    <limit effort="0.0" lower="-3.14" upper="3.14" velocity="0.0"/>
-  </joint>
-  <link name="end_effector_roll_virtual">
-  </link>
-  <joint name="end_effector_yaw_virtual_joint" type="revolute">
-    <parent link="end_effector_roll_virtual"/>
-    <child link="end_effector_yaw_virtual"/>
-    <origin xyz="0 0 0" rpy="0 0 0"/>
-    <axis xyz="0 0 1"/>
-    <limit effort="0.0" lower="-3.14" upper="3.14" velocity="0.0"/>
-  </joint>
-  <link name="end_effector_yaw_virtual">
+    <limit effort="0.0" lower="-3.14" upper="3.14" velocity="1"/>
+  -->
+  </joint>
+  <link name="end_effector_yaw">
+    <visual>
+      <origin xyz="0 0 0" rpy="0 0 0"/>
+      <geometry>
+        <box size="0.01 0.01 0.01"/>
+      </geometry>
+      <material name="end_effector_yaw_material">
+        <color rgba="${green}"/>
+      </material>
+    </visual>
   </link>
   <!-- End effector frame -->
   <joint name="end_effector_joint" type="fixed">
-    <parent link="end_effector_yaw_virtual"/>
+    <parent link="end_effector_yaw"/>
     <child link="end_effector_frame"/>
     <origin xyz="0 0 0" rpy="0 0 0"/>
   </joint>
   <link name="end_effector_frame">
+    <visual>
+      <origin xyz="0 0 0" rpy="0 0 0"/>
+      <geometry>
+        <box size="0.01 0.01 0.01"/>
+      </geometry>
+      <material name="end_effector_roll_material">
+        <color rgba="${green}"/>
+      </material>
+    </visual>
   </link>
   <!-- Gazebo Materials for Arm Links -->
@@ -393,4 +423,10 @@
     <material>Gazebo/Red</material>
   </gazebo>
+  <gazebo reference="end_effector_roll">
+    <material>Gazebo/Green</material>
+  </gazebo>
+  <gazebo reference="end_effector_yaw">
+    <material>Gazebo/Green</material>
+  </gazebo>
   <!-- End effector frame material -->
   <gazebo reference="end_effector_frame">

File: robot_arm/urdf/robot_moveit.urdf.xacro (robot description, xacro)
@@ -11,13 +11,3 @@
     <xacro:include filename="camera.xacro" />
     <xacro:include filename="depth_camera.xacro" />
-    <xacro:include filename="$(find robot_arm)/ros2_control/base_arm_system.ros2_control.xacro" />
-    <xacro:base_arm_system
-        name="base_arm_system" prefix="$(arg prefix)" use_sim_time="$(arg use_sim_time)"
-        use_fake_hardware="$(arg use_fake_hardware)"
-        fake_sensor_commands="$(arg fake_sensor_commands)"/>
-    <gazebo>
-        <plugin name="gazebo_ros2_control" filename="libgazebo_ros2_control.so">
-        <parameters>$(find robot_arm)/config/gazebo_controller_manager.yaml</parameters>
-        </plugin>
-    </gazebo>
 </robot>
