Commit message: Wilson Package Updated

File: wilson/urdf/wilson.urdf.xacro (robot description, xacro)
@@ -6,3 +6,19 @@
     <xacro:arg name="fake_sensor_commands" default="false" />
     <xacro:include filename="wilson_core.xacro" />
+    <xacro:include filename="end_effector.xacro" />
+    <xacro:include filename="wheels.xacro" />
+    <xacro:include filename="lidar.xacro" />
+    <xacro:include filename="camera.xacro" />
+    <xacro:include filename="depth_camera.xacro" />
+    <xacro:include filename="gazebo_references.xacro" />
+    <xacro:include filename="$(find wilson)/ros2_control/wilson_system.ros2_control.xacro" />
+    <xacro:wilson_system
+        name="wilson_system" prefix="$(arg prefix)" use_sim_time="$(arg use_sim_time)"
+        use_fake_hardware="$(arg use_fake_hardware)"
+        fake_sensor_commands="$(arg fake_sensor_commands)"/>
+    <gazebo>
+        <plugin name="gazebo_ros2_control" filename="libgazebo_ros2_control.so">
+        <parameters>$(find wilson)/config/gazebo_controller_manager.yaml</parameters>
+        </plugin>
+    </gazebo>
 </robot>

File: wilson/urdf/wilson_core.xacro (robot description, xacro)
@@ -5,6 +5,8 @@
 <robot xmlns:xacro="http://ros.org/wiki/xacro"
   name="wilson">
-  <link
-    name="base_link">
+  <link name = "base_link">
+  </link>
+  <link
+    name="body_link">
     <inertial>
       <origin
@@ -12,5 +14,5 @@
         rpy="0 0 0" />
       <mass
-        value="7.2003" />
+        value="2" />
       <inertia
         ixx="0.017986"
@@ -27,22 +29,35 @@
       <geometry>
         <mesh
-          filename="package://wilson/meshes/base_link.STL" />
-      </geometry>
-      <material
-        name="">
-        <color
-          rgba="0.79216 0.81961 0.93333 1" />
-      </material>
-    </visual>
-    <collision>
-      <origin
-        xyz="0 0 0"
-        rpy="0 0 0" />
-      <geometry>
-        <mesh
-          filename="package://wilson/meshes/base_link.STL" />
-      </geometry>
-    </collision>
-  </link>
+          filename="package://wilson/meshes/body_link.STL" />
+      </geometry>
+      <material
+        name="">
+        <color
+          rgba="0.3 0.3 0.3 1" />
+      </material>
+    </visual>
+    <collision>
+      <origin
+        xyz="0 0 0"
+        rpy="0 0 0" />
+      <geometry>
+        <mesh
+          filename="package://wilson/collision_meshes/body_link.STL" />
+      </geometry>
+    </collision>
+  </link>
+  <joint
+    name="body_joint"
+    type="fixed">
+    <origin
+      xyz="0 0 0"
+      rpy="0 0 0" />
+    <parent
+      link="base_link" />
+    <child
+      link="body_link" />
+    <axis
+      xyz="0 0 0" />
+  </joint>
   <link
     name="laser_frame">
@@ -72,14 +87,14 @@
         name="">
         <color
-          rgba="0.79216 0.81961 0.93333 1" />
-      </material>
-    </visual>
-    <collision>
-      <origin
-        xyz="0 0 0"
-        rpy="0 0 0" />
-      <geometry>
-        <mesh
-          filename="package://wilson/meshes/laser_frame.STL" />
+          rgba="0.3 0.3 0.3 1" />
+      </material>
+    </visual>
+    <collision>
+      <origin
+        xyz="0 0 0"
+        rpy="0 0 0" />
+      <geometry>
+        <mesh
+          filename="package://wilson/collision_meshes/laser_frame.STL" />
       </geometry>
     </collision>
@@ -92,5 +107,5 @@
       rpy="0 0 0" />
     <parent
-      link="base_link" />
+      link="body_link" />
     <child
       link="laser_frame" />
@@ -129,14 +144,14 @@
         name="">
         <color
-          rgba="0.25098 0.25098 0.25098 1" />
-      </material>
-    </visual>
-    <collision>
-      <origin
-        xyz="0 0 0"
-        rpy="0 0 0" />
-      <geometry>
-        <mesh
-          filename="package://wilson/meshes/camera_link.STL" />
+          rgba="0.3 0.3 0.3 1" />
+      </material>
+    </visual>
+    <collision>
+      <origin
+        xyz="0 0 0"
+        rpy="0 0 0" />
+      <geometry>
+        <mesh
+          filename="package://wilson/collision_meshes/camera_link.STL" />
       </geometry>
     </collision>
@@ -149,5 +164,5 @@
       rpy="0 0 0" />
     <parent
-      link="base_link" />
+      link="body_link" />
     <child
       link="camera_link" />
@@ -182,14 +197,14 @@
         name="">
         <color
-          rgba="0.25098 0.25098 0.25098 1" />
-      </material>
-    </visual>
-    <collision>
-      <origin
-        xyz="0 0 0"
-        rpy="0 0 0" />
-      <geometry>
-        <mesh
-          filename="package://wilson/meshes/depth_camera_link.STL" />
+          rgba="0.3 0.3 0.3 1" />
+      </material>
+    </visual>
+    <collision>
+      <origin
+        xyz="0 0 0"
+        rpy="0 0 0" />
+      <geometry>
+        <mesh
+          filename="package://wilson/collision_meshes/depth_camera_link.STL" />
       </geometry>
     </collision>
@@ -202,5 +217,5 @@
       rpy="0 0 0" />
     <parent
-      link="base_link" />
+      link="body_link" />
     <child
       link="depth_camera_link" />
@@ -215,12 +230,12 @@
         rpy="0 0 0" />
       <mass
-        value="0" />
-      <inertia
-        ixx="0"
-        ixy="0"
-        ixz="0"
-        iyy="0"
-        iyz="0"
-        izz="0" />
+        value="0.1" />
+      <inertia
+        ixx="0.001"
+        ixy="0.001"
+        ixz="0.001"
+        iyy="0.001"
+        iyz="0.001"
+        izz="0.001" />
     </inertial>
     <visual>
@@ -235,14 +250,14 @@
         name="">
         <color
-          rgba="1 1 1 1" />
-      </material>
-    </visual>
-    <collision>
-      <origin
-        xyz="0 0 0"
-        rpy="0 0 0" />
-      <geometry>
-        <mesh
-          filename="package://wilson/meshes/link_1.STL" />
+          rgba="0.3 0.3 0.3 1" />
+      </material>
+    </visual>
+    <collision>
+      <origin
+        xyz="0 0 0"
+        rpy="0 0 0" />
+      <geometry>
+        <mesh
+          filename="package://wilson/collision_meshes/link_1.STL" />
       </geometry>
     </collision>
@@ -255,5 +270,5 @@
       rpy="0 0 0" />
     <parent
-      link="base_link" />
+      link="body_link" />
     <child
       link="link_1" />
@@ -263,6 +278,6 @@
       lower="-2.3562"
       upper="2.3562"
-      effort="0"
-      velocity="0" />
+      effort="100"
+      velocity="1.0" />
   </joint>
   <link
@@ -293,14 +308,14 @@
         name="">
         <color
-          rgba="0.79216 0.81961 0.93333 1" />
-      </material>
-    </visual>
-    <collision>
-      <origin
-        xyz="0 0 0"
-        rpy="0 0 0" />
-      <geometry>
-        <mesh
-          filename="package://wilson/meshes/link_2.STL" />
+          rgba="0.3 0.3 0.3 1" />
+      </material>
+    </visual>
+    <collision>
+      <origin
+        xyz="0 0 0"
+        rpy="0 0 0" />
+      <geometry>
+        <mesh
+          filename="package://wilson/collision_meshes/link_2.STL" />
       </geometry>
     </collision>
@@ -317,10 +332,10 @@
       link="link_2" />
     <axis
-      xyz="0 0 -1" />
+      xyz="0 0 1" />
     <limit
       lower="-2.3562"
       upper="2.3562"
-      effort="0"
-      velocity="0" />
+      effort="100"
+      velocity="1.0" />
   </joint>
   <link
@@ -351,14 +366,14 @@
         name="">
         <color
-          rgba="0.79216 0.81961 0.93333 1" />
-      </material>
-    </visual>
-    <collision>
-      <origin
-        xyz="0 0 0"
-        rpy="0 0 0" />
-      <geometry>
-        <mesh
-          filename="package://wilson/meshes/link_3.STL" />
+          rgba="0.3 0.3 0.3 1" />
+      </material>
+    </visual>
+    <collision>
+      <origin
+        xyz="0 0 0"
+        rpy="0 0 0" />
+      <geometry>
+        <mesh
+          filename="package://wilson/collision_meshes/link_3.STL" />
       </geometry>
     </collision>
@@ -375,10 +390,10 @@
       link="link_3" />
     <axis
-      xyz="0 0 -1" />
+      xyz="0 0 1" />
     <limit
       lower="-2.3562"
       upper="2.3562"
-      effort="0"
-      velocity="0" />
+      effort="100"
+      velocity="1.0" />
   </joint>
   <link
@@ -409,14 +424,14 @@
         name="">
         <color
-          rgba="0.79216 0.81961 0.93333 1" />
-      </material>
-    </visual>
-    <collision>
-      <origin
-        xyz="0 0 0"
-        rpy="0 0 0" />
-      <geometry>
-        <mesh
-          filename="package://wilson/meshes/link_4.STL" />
+          rgba="0.3 0.3 0.3 1" />
+      </material>
+    </visual>
+    <collision>
+      <origin
+        xyz="0 0 0"
+        rpy="0 0 0" />
+      <geometry>
+        <mesh
+          filename="package://wilson/collision_meshes/link_4.STL" />
       </geometry>
     </collision>
@@ -433,10 +448,10 @@
       link="link_4" />
     <axis
-      xyz="0 0 -1" />
+      xyz="0 0 1" />
     <limit
       lower="-2.3562"
       upper="2.3562"
-      effort="0"
-      velocity="0" />
+      effort="100"
+      velocity="1.0" />
   </joint>
   <link
@@ -467,14 +482,14 @@
         name="">
         <color
-          rgba="0.25098 0.25098 0.25098 1" />
-      </material>
-    </visual>
-    <collision>
-      <origin
-        xyz="0 0 0"
-        rpy="0 0 0" />
-      <geometry>
-        <mesh
-          filename="package://wilson/meshes/gripper_base.STL" />
+          rgba="0.3 0.3 0.3 1" />
+      </material>
+    </visual>
+    <collision>
+      <origin
+        xyz="0 0 0"
+        rpy="0 0 0" />
+      <geometry>
+        <mesh
+          filename="package://wilson/collision_meshes/gripper_base.STL" />
       </geometry>
     </collision>
@@ -520,14 +535,14 @@
         name="">
         <color
-          rgba="0.25098 0.25098 0.25098 1" />
-      </material>
-    </visual>
-    <collision>
-      <origin
-        xyz="0 0 0"
-        rpy="0 0 0" />
-      <geometry>
-        <mesh
-          filename="package://wilson/meshes/gripper_left_finger.STL" />
+          rgba="0.3 0.3 0.3 1" />
+      </material>
+    </visual>
+    <collision>
+      <origin
+        xyz="0 0 0"
+        rpy="0 0 0" />
+      <geometry>
+        <mesh
+          filename="package://wilson/collision_meshes/gripper_left_finger.STL" />
       </geometry>
     </collision>
@@ -578,14 +593,14 @@
         name="">
         <color
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