Commit message: Wilson Moveit Config Added

File: wilson/ros2_control/wilson_system.ros2_control.xacro (robot description, xacro)
@@ -108,5 +108,5 @@
         </command_interface>
         <state_interface name="position">
-          <param name="initial_value">${-pi/2}</param>
+          <param name="initial_value">0.0</param>
         </state_interface>
         <state_interface name="velocity">

File: wilson/urdf/wheels.xacro (robot description, xacro)
@@ -81,5 +81,5 @@
         <parent link="body_link"/>
         <child link="front_caster_wheel"/>
-        <origin xyz=".18 0.0 -0.01"/>
+        <origin xyz=".21 0.0 -0.01"/>
     </joint>
     <link name="front_caster_wheel">

File: wilson/urdf/wilson_core.xacro (robot description, xacro)
@@ -14,5 +14,5 @@
         rpy="0 0 0" />
       <mass
-        value="2" />
+        value="3" />
       <inertia
         ixx="0.017986"
@@ -67,5 +67,5 @@
         rpy="0 0 0" />
       <mass
-        value="0.041194" />
+        value="0.001" />
       <inertia
         ixx="5.4479E-06"
@@ -112,8 +112,4 @@
     <axis
       xyz="0 0 0" />
-    <mimic
-      joint="gripper_left_finger_joint"
-      multiplier="1"
-      offset="0" />
   </joint>
   <link
@@ -230,5 +226,5 @@
         rpy="0 0 0" />
       <mass
-        value="0.1" />
+        value="0.001" />
       <inertia
         ixx="0.001"
@@ -288,5 +284,5 @@
         rpy="0 0 0" />
       <mass
-        value="0.092908" />
+        value="0.001" />
       <inertia
         ixx="1.8027E-05"
@@ -346,5 +342,5 @@
         rpy="0 0 0" />
       <mass
-        value="0.04259" />
+        value="0.001" />
       <inertia
         ixx="1.0479E-05"
@@ -404,5 +400,5 @@
         rpy="0 0 0" />
       <mass
-        value="0.088822" />
+        value="0.0001" />
       <inertia
         ixx="5.9516E-05"
@@ -462,5 +458,5 @@
         rpy="0 0 0" />
       <mass
-        value="0.1047" />
+        value="0.001" />
       <inertia
         ixx="0.00012973"
@@ -515,5 +511,5 @@
         rpy="0 0 0" />
       <mass
-        value="0.02298" />
+        value="0.001" />
       <inertia
         ixx="6.2762E-06"
@@ -573,5 +569,5 @@
         rpy="0 0 0" />
       <mass
-        value="0.02298" />
+        value="0.001" />
       <inertia
         ixx="6.2762E-06"
@@ -619,5 +615,5 @@
       xyz="0 0 1" />
     <limit
-      lower="0"
+      lower="-0.05"
       upper="0"
       effort="0"
